File: kicad/jelly.sch (KiCad schematic (older format))
At the start: 35 parts, among them M1 PAGER_MOTOR, M2 PAGER_MOTOR, P1 CONN_01X01, P10 CONN_01X01, P11 CONN_01X01, P12 CONN_01X01, P13 CONN_01X01, P14 CONN_01X01, P15 CONN_01X01, P2 CONN_01X01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

Commit message: Add logo and name
Parts:
- added DNP4: logo, custom:logo, symbol placeholder
- added DNP5: name, custom:name, symbol placeholder
Changed lines of the file:
@@
 $EndComp
 $Comp
-L GND-RESCUE-bristle_bot #PWR01
+L GND-RESCUE-bristle_bot #PWR2
 U 1 1 57C0D38E
 P 1325 3225
-F 0 "#PWR01" H 1325 3225 30  0001 C CNN
+F 0 "#PWR2" H 1325 3225 30  0001 C CNN
 F 1 "GND" H 1325 3155 30  0001 C CNN
 F 2 "" H 1325 3225 60  0000 C CNN
@@
 $EndComp
 $Comp
-L VCC #PWR02
+L VCC #PWR1
 U 1 1 57C0D391
 P 1325 1275
-F 0 "#PWR02" H 1325 1375 30  0001 C CNN
+F 0 "#PWR1" H 1325 1375 30  0001 C CNN
 F 1 "VCC" H 1325 1375 30  0000 C CNN
 F 2 "" H 1325 1275 60  0001 C CNN
@@
 $EndComp
 $Comp
-L VCC #PWR03
+L VCC #PWR5
 U 1 1 57C0D393
 P 4200 2900
-F 0 "#PWR03" H 4200 3000 30  0001 C CNN
+F 0 "#PWR5" H 4200 3000 30  0001 C CNN
 F 1 "VCC" H 4200 3000 30  0000 C CNN
 F 2 "" H 4200 2900 60  0001 C CNN
@@
 $EndComp
 $Comp
-L VCC #PWR04
+L VCC #PWR8
 U 1 1 57C0D394
 P 5200 2650
-F 0 "#PWR04" H 5200 2750 30  0001 C CNN
+F 0 "#PWR8" H 5200 2750 30  0001 C CNN
 F 1 "VCC" H 5200 2750 30  0000 C CNN
 F 2 "" H 5200 2650 60  0001 C CNN
@@
 $EndComp
 $Comp
-L VCC #PWR05
+L VCC #PWR14
 U 1 1 57C0D397
 P 8150 2550
-F 0 "#PWR05" H 8150 2650 30  0001 C CNN
+F 0 "#PWR14" H 8150 2650 30  0001 C CNN
 F 1 "VCC" H 8150 2650 30  0000 C CNN
 F 2 "" H 8150 2550 60  0001 C CNN
@@
 $EndComp
 $Comp
-L VCC #PWR06
+L VCC #PWR11
 U 1 1 57C0D39B
 P 7150 2800
-F 0 "#PWR06" H 7150 2900 30  0001 C CNN
+F 0 "#PWR11" H 7150 2900 30  0001 C CNN
 F 1 "VCC" H 7150 2900 30  0000 C CNN
 F 2 "" H 7150 2800 60  0001 C CNN
@@
 $EndComp
 $Comp
-L VCC #PWR07
+L VCC #PWR18
 U 1 1 57C0D3A1
 P 9500 2600
-F 0 "#PWR07" H 9500 2700 30  0001 C CNN
+F 0 "#PWR18" H 9500 2700 30  0001 C CNN
 F 1 "VCC" H 9500 2700 30  0000 C CNN
 F 2 "" H 9500 2600 60  0001 C CNN
@@
 $EndComp
 $Comp
-L VCC #PWR08
+L VCC #PWR10
 U 1 1 57C0D3A4
 P 6800 2700
-F 0 "#PWR08" H 6800 2800 30  0001 C CNN
+F 0 "#PWR10" H 6800 2800 30  0001 C CNN
 F 1 "VCC" H 6800 2800 30  0000 C CNN
 F 2 "" H 6800 2700 60  0001 C CNN
@@
 $EndComp
 $Comp
-L VCC #PWR09
+L VCC #PWR3
 U 1 1 57C0D3B0
 P 1450 4350
-F 0 "#PWR09" H 1450 4450 30  0001 C CNN
+F 0 "#PWR3" H 1450 4450 30  0001 C CNN
 F 1 "VCC" H 1450 4450 30  0000 C CNN
 F 2 "" H 1450 4350 60  0001 C CNN
@@
 $EndComp
 $Comp
-L VCC #PWR010
+L VCC #PWR13
 U 1 1 57C309E3
 P 7900 4600
-F 0 "#PWR010" H 7900 4700 30  0001 C CNN
+F 0 "#PWR13" H 7900 4700 30  0001 C CNN
 F 1 "VCC" H 7900 4700 30  0000 C CNN
 F 2 "" H 7900 4600 60  0001 C CNN
@@
 Vout2
 $Comp
-L GND-RESCUE-bristle_bot #PWR011
+L GND-RESCUE-bristle_bot #PWR6
 U 1 1 57C36163
 P 4600 4550
-F 0 "#PWR011" H 4600 4550 30  0001 C CNN
+F 0 "#PWR6" H 4600 4550 30  0001 C CNN
 F 1 "GND" H 4600 4480 30  0001 C CNN
 F 2 "" H 4600 4550 60  0001 C CNN
@@
 $EndComp
 $Comp
-L VCC #PWR012
+L VCC #PWR17
 U 1 1 57C3486C
 P 8450 6350
-F 0 "#PWR012" H 8450 6450 30  0001 C CNN
+F 0 "#PWR17" H 8450 6450 30  0001 C CNN
 F 1 "VCC" H 8450 6450 30  0000 C CNN
 F 2 "" H 8450 6350 60  0001 C CNN
@@
 $EndComp
 $Comp
-L GND #PWR013
+L GND #PWR9
 U 1 1 57EC11E5
 P 5350 3175
-F 0 "#PWR013" H 5350 2925 50  0001 C CNN
+F 0 "#PWR9" H 5350 2925 50  0001 C CNN
 F 1 "GND" H 5355 3002 50  0000 C CNN
 F 2 "" H 5350 3175 50  0000 C CNN
@@
 $EndComp
 $Comp
-L GND #PWR014
+L GND #PWR16
 U 1 1 57EC1326
 P 8325 3075
-F 0 "#PWR014" H 8325 2825 50  0001 C CNN
+F 0 "#PWR16" H 8325 2825 50  0001 C CNN
 F 1 "GND" H 8330 2902 50  0000 C CNN
 F 2 "" H 8325 3075 50  0000 C CNN
@@
 $EndComp
 $Comp
-L GND #PWR015
+L GND #PWR7
 U 1 1 57EC1A42
 P 5175 3500
-F 0 "#PWR015" H 5175 3250 50  0001 C CNN
+F 0 "#PWR7" H 5175 3250 50  0001 C CNN
 F 1 "GND" H 5180 3327 50  0000 C CNN
 F 2 "" H 5175 3500 50  0000 C CNN
@@
 $EndComp
 $Comp
-L GND #PWR016
+L GND #PWR15
 U 1 1 57EC1E47
 P 8225 3475
-F 0 "#PWR016" H 8225 3225 50  0001 C CNN
+F 0 "#PWR15" H 8225 3225 50  0001 C CNN
 F 1 "GND" H 8230 3302 50  0000 C CNN
 F 2 "" H 8225 3475 50  0000 C CNN
@@
 Connection ~ 2225 3000
 $Comp
-L GND-RESCUE-bristle_bot #PWR017
+L GND-RESCUE-bristle_bot #PWR4
 U 1 1 57EC6243
 P 2225 3575
-F 0 "#PWR017" H 2225 3575 30  0001 C CNN
+F 0 "#PWR4" H 2225 3575 30  0001 C CNN
 F 1 "GND" H 2225 3505 30  0001 C CNN
 F 2 "" H 2225 3575 60  0000 C CNN
@@
 	1325 2700 1325 2025
 $Comp
-L GND-RESCUE-bristle_bot #PWR?
+L GND-RESCUE-bristle_bot #PWR12
 U 1 1 57F92FC8
 P 7800 6275
-F 0 "#PWR?" H 7800 6275 30  0001 C CNN
+F 0 "#PWR12" H 7800 6275 30  0001 C CNN
 F 1 "GND" H 7800 6205 30  0001 C CNN
 F 2 "" H 7800 6275 60  0000 C CNN
@@
 Wire Wire Line
 	7800 6200 7800 6275
+$Comp
+L placeholder DNP4
+U 1 1 580214C3
+P 9900 6200
+F 0 "DNP4" H 9900 6350 60  0000 C CNN
+F 1 "logo" H 9900 6450 60  0000 C CNN
+F 2 "custom:logo" H 9900 6350 60  0001 C CNN
+F 3 "" H 9900 6350 60  0001 C CNN
+	1    9900 6200
+	1    0    0    -1
+$EndComp
+$Comp
+L placeholder DNP5
+U 1 1 5802487F
+P 10350 6175
+F 0 "DNP5" H 10350 6325 60  0000 C CNN
+F 1 "name" H 10350 6425 60  0000 C CNN
+F 2 "custom:name" H 10350 6325 60  0001 C CNN
+F 3 "" H 10350 6325 60  0001 C CNN
+	1    10350 6175
+	1    0    0    -1
+$EndComp
 $EndSCHEMATC

Commit message: Make image for LDR silkscreen
Parts:
- DNP3: footprint custom:ldr_image -> custom:ldr_image_flipped
Changed lines of the file:
@@
 $EndComp
 $Comp
-L GND-RESCUE-bristle_bot #PWR2
+L GND-RESCUE-bristle_bot #PWR01
 U 1 1 57C0D38E
 P 1325 3225
-F 0 "#PWR2" H 1325 3225 30  0001 C CNN
+F 0 "#PWR01" H 1325 3225 30  0001 C CNN
 F 1 "GND" H 1325 3155 30  0001 C CNN
 F 2 "" H 1325 3225 60  0000 C CNN
@@
 $EndComp
 $Comp
-L VCC #PWR1
+L VCC #PWR02
 U 1 1 57C0D391
 P 1325 1275
-F 0 "#PWR1" H 1325 1375 30  0001 C CNN
+F 0 "#PWR02" H 1325 1375 30  0001 C CNN
 F 1 "VCC" H 1325 1375 30  0000 C CNN
 F 2 "" H 1325 1275 60  0001 C CNN
@@
 $EndComp
 $Comp
-L VCC #PWR5
+L VCC #PWR03
 U 1 1 57C0D393
 P 4200 2900
-F 0 "#PWR5" H 4200 3000 30  0001 C CNN
+F 0 "#PWR03" H 4200 3000 30  0001 C CNN
 F 1 "VCC" H 4200 3000 30  0000 C CNN
 F 2 "" H 4200 2900 60  0001 C CNN
@@
 $EndComp
 $Comp
-L VCC #PWR8
+L VCC #PWR04
 U 1 1 57C0D394
 P 5200 2650
-F 0 "#PWR8" H 5200 2750 30  0001 C CNN
+F 0 "#PWR04" H 5200 2750 30  0001 C CNN
 F 1 "VCC" H 5200 2750 30  0000 C CNN
 F 2 "" H 5200 2650 60  0001 C CNN
@@
 $EndComp
 $Comp
-L VCC #PWR14
+L VCC #PWR05
 U 1 1 57C0D397
 P 8150 2550
-F 0 "#PWR14" H 8150 2650 30  0001 C CNN
+F 0 "#PWR05" H 8150 2650 30  0001 C CNN
 F 1 "VCC" H 8150 2650 30  0000 C CNN
 F 2 "" H 8150 2550 60  0001 C CNN
@@
 $EndComp
 $Comp
-L VCC #PWR11
+L VCC #PWR06
 U 1 1 57C0D39B
 P 7150 2800
-F 0 "#PWR11" H 7150 2900 30  0001 C CNN
+F 0 "#PWR06" H 7150 2900 30  0001 C CNN
 F 1 "VCC" H 7150 2900 30  0000 C CNN
 F 2 "" H 7150 2800 60  0001 C CNN
@@
 $EndComp
 $Comp
-L VCC #PWR18
+L VCC #PWR07
 U 1 1 57C0D3A1
 P 9500 2600
-F 0 "#PWR18" H 9500 2700 30  0001 C CNN
+F 0 "#PWR07" H 9500 2700 30  0001 C CNN
 F 1 "VCC" H 9500 2700 30  0000 C CNN
 F 2 "" H 9500 2600 60  0001 C CNN
@@
 $EndComp
 $Comp
-L VCC #PWR10
+L VCC #PWR08
 U 1 1 57C0D3A4
 P 6800 2700
-F 0 "#PWR10" H 6800 2800 30  0001 C CNN
+F 0 "#PWR08" H 6800 2800 30  0001 C CNN
 F 1 "VCC" H 6800 2800 30  0000 C CNN
 F 2 "" H 6800 2700 60  0001 C CNN
@@
 $EndComp
 $Comp
-L VCC #PWR3
+L VCC #PWR09
 U 1 1 57C0D3B0
 P 1450 4350
-F 0 "#PWR3" H 1450 4450 30  0001 C CNN
+F 0 "#PWR09" H 1450 4450 30  0001 C CNN
 F 1 "VCC" H 1450 4450 30  0000 C CNN
 F 2 "" H 1450 4350 60  0001 C CNN
@@
 $EndComp
 $Comp
-L VCC #PWR13
+L VCC #PWR010
 U 1 1 57C309E3
 P 7900 4600
-F 0 "#PWR13" H 7900 4700 30  0001 C CNN
+F 0 "#PWR010" H 7900 4700 30  0001 C CNN
 F 1 "VCC" H 7900 4700 30  0000 C CNN
 F 2 "" H 7900 4600 60  0001 C CNN
@@
 F 0 "DNP3" H 9350 6350 60  0000 C CNN
 F 1 "ldr_image" H 9350 6450 60  0000 C CNN
-F 2 "custom:ldr_image" H 9350 6350 60  0001 C CNN
+F 2 "custom:ldr_image_flipped" H 9350 6350 60  0001 C CNN
 F 3 "" H 9350 6350 60  0001 C CNN
 	1    9350 6200
@@
 Vout2
 $Comp
-L GND-RESCUE-bristle_bot #PWR6
+L GND-RESCUE-bristle_bot #PWR011
 U 1 1 57C36163
 P 4600 4550
-F 0 "#PWR6" H 4600 4550 30  0001 C CNN
+F 0 "#PWR011" H 4600 4550 30  0001 C CNN
 F 1 "GND" H 4600 4480 30  0001 C CNN
 F 2 "" H 4600 4550 60  0001 C CNN
@@
 $EndComp
 $Comp
-L VCC #PWR17
+L VCC #PWR012
 U 1 1 57C3486C
 P 8450 6350
-F 0 "#PWR17" H 8450 6450 30  0001 C CNN
+F 0 "#PWR012" H 8450 6450 30  0001 C CNN
 F 1 "VCC" H 8450 6450 30  0000 C CNN
 F 2 "" H 8450 6350 60  0001 C CNN
@@
 $EndComp
 $Comp
-L GND #PWR9
+L GND #PWR013
 U 1 1 57EC11E5
 P 5350 3175
-F 0 "#PWR9" H 5350 2925 50  0001 C CNN
+F 0 "#PWR013" H 5350 2925 50  0001 C CNN
 F 1 "GND" H 5355 3002 50  0000 C CNN
 F 2 "" H 5350 3175 50  0000 C CNN
@@
 $EndComp
 $Comp
-L GND #PWR16
+L GND #PWR014
 U 1 1 57EC1326
 P 8325 3075
-F 0 "#PWR16" H 8325 2825 50  0001 C CNN
+F 0 "#PWR014" H 8325 2825 50  0001 C CNN
 F 1 "GND" H 8330 2902 50  0000 C CNN
 F 2 "" H 8325 3075 50  0000 C CNN
@@
 $EndComp
 $Comp
-L GND #PWR7
+L GND #PWR015
 U 1 1 57EC1A42
 P 5175 3500
-F 0 "#PWR7" H 5175 3250 50  0001 C CNN
+F 0 "#PWR015" H 5175 3250 50  0001 C CNN
 F 1 "GND" H 5180 3327 50  0000 C CNN
 F 2 "" H 5175 3500 50  0000 C CNN
@@
 $EndComp
 $Comp
-L GND #PWR15
+L GND #PWR016
 U 1 1 57EC1E47
 P 8225 3475
-F 0 "#PWR15" H 8225 3225 50  0001 C CNN
+F 0 "#PWR016" H 8225 3225 50  0001 C CNN
 F 1 "GND" H 8230 3302 50  0000 C CNN
 F 2 "" H 8225 3475 50  0000 C CNN
@@
 Connection ~ 2225 3000
 $Comp
-L GND-RESCUE-bristle_bot #PWR4
+L GND-RESCUE-bristle_bot #PWR017
 U 1 1 57EC6243
 P 2225 3575
-F 0 "#PWR4" H 2225 3575 30  0001 C CNN
+F 0 "#PWR017" H 2225 3575 30  0001 C CNN
 F 1 "GND" H 2225 3505 30  0001 C CNN
 F 2 "" H 2225 3575 60  0000 C CNN
@@
 	1325 2700 1325 2025
 $Comp
-L GND-RESCUE-bristle_bot #PWR12
+L GND-RESCUE-bristle_bot #PWR018
 U 1 1 57F92FC8
 P 7800 6275
-F 0 "#PWR12" H 7800 6275 30  0001 C CNN
+F 0 "#PWR018" H 7800 6275 30  0001 C CNN
 F 1 "GND" H 7800 6205 30  0001 C CNN
 F 2 "" H 7800 6275 60  0000 C CNN

Commit message: Add resistor silkscreen
Parts:
- added DNP6: resistor_R1, custom:resistor, symbol placeholder
- added DNP7: resistor_R2, custom:resistor, symbol placeholder
- added DNP8: resistor_R3, custom:resistor, symbol placeholder
- added DNP9: resistor_R4, custom:resistor, symbol placeholder
- R1, R2, R3, R4: footprint KiCad/Discret.pretty:R3-5 -> custom:R3-5
Changed lines of the file:
@@
 F 0 "R4" V 9280 2600 40  0000 C CNN
 F 1 "120" V 9207 2601 40  0000 C CNN
-F 2 "KiCad/Discret.pretty:R3-5" V 9130 2600 30  0001 C CNN
+F 2 "custom:R3-5" V 9130 2600 30  0001 C CNN
 F 3 "~" H 9200 2600 30  0000 C CNN
 	1    9200 2600
@@
 F 0 "R2" V 6580 2700 40  0000 C CNN
 F 1 "120" V 6507 2701 40  0000 C CNN
-F 2 "KiCad/Discret.pretty:R3-5" V 6430 2700 30  0001 C CNN
+F 2 "custom:R3-5" V 6430 2700 30  0001 C CNN
 F 3 "~" H 6500 2700 30  0000 C CNN
 	1    6500 2700
@@
 F 0 "R1" H 2295 2821 50  0000 L CNN
 F 1 "1k" H 2295 2730 50  0000 L CNN
-F 2 "KiCad/Discret.pretty:R3-5" V 2155 2775 50  0001 C CNN
+F 2 "custom:R3-5" V 2155 2775 50  0001 C CNN
 F 3 "" H 2225 2775 50  0000 C CNN
 	1    2225 2775
@@
 F 0 "R3" H 2295 3296 50  0000 L CNN
 F 1 "100k" H 2295 3205 50  0000 L CNN
-F 2 "KiCad/Discret.pretty:R3-5" V 2155 3250 50  0001 C CNN
+F 2 "custom:R3-5" V 2155 3250 50  0001 C CNN
 F 3 "" H 2225 3250 50  0000 C CNN
 	1    2225 3250
@@
 	1    0    0    -1
 $EndComp
+$Comp
+L placeholder DNP6
+U 1 1 58028D21
+P 9050 5100
+F 0 "DNP6" H 9050 5250 60  0000 C CNN
+F 1 "resistor_R1" H 9050 5350 60  0000 C CNN
+F 2 "custom:resistor" H 9050 5250 60  0001 C CNN
+F 3 "" H 9050 5250 60  0001 C CNN
+	1    9050 5100
+	1    0    0    -1
+$EndComp
+$Comp
+L placeholder DNP7
+U 1 1 58028E57
+P 9600 5125
+F 0 "DNP7" H 9600 5275 60  0000 C CNN
+F 1 "resistor_R2" H 9600 5375 60  0000 C CNN
+F 2 "custom:resistor" H 9600 5275 60  0001 C CNN
+F 3 "" H 9600 5275 60  0001 C CNN
+	1    9600 5125
+	1    0    0    -1
+$EndComp
+$Comp
+L placeholder DNP8
+U 1 1 58028EEE
+P 10125 5150
+F 0 "DNP8" H 10125 5300 60  0000 C CNN
+F 1 "resistor_R3" H 10125 5400 60  0000 C CNN
+F 2 "custom:resistor" H 10125 5300 60  0001 C CNN
+F 3 "" H 10125 5300 60  0001 C CNN
+	1    10125 5150
+	1    0    0    -1
+$EndComp
+$Comp
+L placeholder DNP9
+U 1 1 58029990
+P 10675 5100
+F 0 "DNP9" H 10675 5250 60  0000 C CNN
+F 1 "resistor_R4" H 10675 5350 60  0000 C CNN
+F 2 "custom:resistor" H 10675 5250 60  0001 C CNN
+F 3 "" H 10675 5250 60  0001 C CNN
+	1    10675 5100
+	1    0    0    -1
+$EndComp
